Commit message: updates to urdf

File: source/humanoid_assets/data/urdf/t1/t1.urdf (robot description, URDF)
Before this commit: robot T1, 24 links, 23 joints
Joints:
- joint joint_al4: origin xyz=0 0.1471 0 rpy=0 0 0 -> xyz=0 0.1471 0 rpy=0 0 -1.5707
- joint joint_ar4: axis 0 0 1 -> 0 0 -1; origin xyz=0 -0.1471 0 rpy=0 0 0 -> xyz=0 -0.1471 0 rpy=0 0 1.5707

Commit message: update booster to match deployment values. Add debug viz to replay

File: source/humanoid_assets/data/urdf/t1/t1.urdf (robot description, URDF)
Before this commit: robot T1, 24 links, 23 joints
Joints:
- joint joint_al3: axis 0 1 0 -> 0 -1 0

Commit message: recreate booster gym training

File: source/humanoid_assets/data/urdf/t1/t1.urdf (robot description, URDF)
Before this commit: robot T1, 24 links, 23 joints
Joints:
- joint joint_al2: origin xyz=0 0.047 0 rpy=-1.45 0 0 -> xyz=0 0.047 0 rpy=0 0 0
- joint joint_ar2: origin xyz=0 -0.047 0 rpy=1.45 0 0 -> xyz=0 -0.047 0 rpy=0 0 0
